Commit message: initial commit

File: src/rrbot_description/urdf/gazebo_plugins.xacro (robot description, xacro)
@@ -1,67 +1,4 @@
 <?xml version="1.0"?>
 <robot xmlns:xacro="http://www.ros.org/wiki/xacro" name="rrbot">
-  <!-- ros_control plugin -->
-  <gazebo>
-    <plugin name="gazebo_ros_control" filename="libgazebo_ros_control.so">
-      <robotNamespace>/rrbot</robotNamespace>
-      <robotSimType>gazebo_ros_control/DefaultRobotHWSim</robotSimType>
-    </plugin>
-  </gazebo>
-  <transmission name="tran1">
-    <type>transmission_interface/SimpleTransmission</type>
-    <joint name="joint1">
-      <hardwareInterface>hardware_interface/EffortJointInterface</hardwareInterface>
-    </joint>
-    <actuator name="motor1">
-      <hardwareInterface>hardware_interface/EffortJointInterface</hardwareInterface>
-      <mechanicalReduction>1</mechanicalReduction>
-    </actuator>
-  </transmission>
-  <transmission name="tran2">
-    <type>transmission_interface/SimpleTransmission</type>
-    <joint name="joint2">
-      <hardwareInterface>hardware_interface/EffortJointInterface</hardwareInterface>
-    </joint>
-    <actuator name="motor2">
-      <hardwareInterface>hardware_interface/EffortJointInterface</hardwareInterface>
-      <mechanicalReduction>1</mechanicalReduction>
-    </actuator>
-  </transmission>
-  <!-- hokuyo -->
-  <gazebo reference="hokuyo_link">
-    <sensor type="ray" name="head_hokuyo_sensor">
-      <pose>0 0 0 0 0 0</pose>
-      <visualize>true</visualize>
-      <update_rate>40</update_rate>
-      <ray>
-        <scan>
-          <horizontal>
-            <samples>720</samples>
-            <resolution>1</resolution>
-            <min_angle>-3.14159</min_angle>
-            <max_angle>3.14159</max_angle>
-          </horizontal>
-        </scan>
-        <range>
-          <min>0.10</min>
-          <max>30.0</max>
-          <resolution>0.01</resolution>
-        </range>
-        <noise>
-          <type>gaussian</type>
-          <!-- Noise parameters based on published spec for Hokuyo laser
-               achieving "+-30mm" accuracy at range < 10m.  A mean of 0.0m and
-               stddev of 0.01m will put 99.7% of samples within 0.03m of the true
-               reading. -->
-          <mean>0.0</mean>
-          <stddev>0.01</stddev>
-        </noise>
-      </ray>
-      <plugin name="gazebo_ros_head_hokuyo_controller" filename="libgazebo_ros_laser.so">
-        <topicName>/rrbot/laser/scan</topicName>
-        <frameName>hokuyo_link</frameName>
-      </plugin>
-    </sensor>
-  </gazebo>
   <!-- camera -->
   <gazebo reference="camera_link">

File: src/rrbot_description/urdf/gazebo_properties.xacro (robot description, xacro)
@@ -7,5 +7,5 @@
   <!-- Link2 -->
   <gazebo reference="link2">
-    <material>Gazebo/Black</material>
+    <material>Gazebo/Orange</material>
   </gazebo>
   <!-- Link3 -->

File: src/rrbot_description/urdf/rrbot.xacro (robot description, xacro)
@@ -54,5 +54,5 @@
 	<box size="${width} ${width} ${height2}"/>
       </geometry>
-      <material name="black"/>
+      <material name="orange"/>
     </visual>
     <inertial>
@@ -90,34 +90,8 @@
     </inertial>
   </link>
-  <joint name="hokuyo_joint" type="fixed">
-    <axis xyz="0 1 0" />
-    <origin xyz="0 0 ${height3 - axel_offset/2}" rpy="0 0 0"/>
-    <parent link="link3"/>
-    <child link="hokuyo_link"/>
-  </joint>
-  <!-- Hokuyo Laser -->
-  <link name="hokuyo_link">
-    <collision>
-      <origin xyz="0 0 0" rpy="0 0 0"/>
-      <geometry>
-	<box size="0.1 0.1 0.1"/>
-      </geometry>
-    </collision>
-    <visual>
-      <origin xyz="0 0 0" rpy="0 0 0"/>
-      <geometry>
-        <mesh filename="package://rrbot_description/meshes/hokuyo.dae"/>
-      </geometry>
-    </visual>
-    <inertial>
-      <mass value="1e-5" />
-      <origin xyz="0 0 0" rpy="0 0 0"/>
-      <inertia ixx="1e-6" ixy="0" ixz="0" iyy="1e-6" iyz="0" izz="1e-6" />
-    </inertial>
-  </link>
   <joint name="camera_joint" type="fixed">
     <axis xyz="0 1 0" />
     <origin xyz="${camera_link} 0 ${height3 - axel_offset*2}" rpy="0 0 0"/>
-    <parent link="link3"/>
+    <parent link="link1"/>
     <child link="camera_link"/>
   </joint>
@@ -125,5 +99,5 @@
   <link name="camera_link">
     <collision>
-      <origin xyz="0 0 0" rpy="0 0 0"/>
+      <origin xyz="0 0 ${height2}" rpy="0 0.5 0"/>
       <geometry>
 	<box size="${camera_link} ${camera_link} ${camera_link}"/>
@@ -131,5 +105,5 @@
     </collision>
     <visual>
-      <origin xyz="0 0 0" rpy="0 0 0"/>
+      <origin xyz="0 0 ${height2}" rpy="0 0.5 0"/>
       <geometry>
 	<box size="${camera_link} ${camera_link} ${camera_link}"/>
@@ -139,5 +113,5 @@
     <inertial>
       <mass value="1e-5" />
-      <origin xyz="0 0 0" rpy="0 0 0"/>
+      <origin xyz="0 0 ${height2}" rpy="0 0.5 0"/>
       <inertia ixx="1e-6" ixy="0" ixz="0" iyy="1e-6" iyz="0" izz="1e-6" />
     </inertial>

Commit message: changed rrbot to be simpler and better looking

File: src/rrbot_description/urdf/gazebo_plugins.xacro (robot description, xacro)
@@ -48,11 +48,3 @@
     </sensor>
   </gazebo>
-  <!-- Joint state publisher plugin -->
-  <gazebo>
-    <plugin name="joint_state_publisher" filename="libgazebo_ros_joint_state_publisher.so">
-        <robotNamespace>rrbot</robotNamespace>
-        <jointName>joint1, joint2</jointName>
-        <updateRate>100</updateRate>
-    </plugin>
-  </gazebo>
 </robot>

File: src/rrbot_description/urdf/rrbot.xacro (robot description, xacro)
@@ -5,5 +5,4 @@
   <xacro:include filename="$(find rrbot_description)/urdf/materials.xacro"/>
   <xacro:include filename="$(find rrbot_description)/urdf/gazebo_properties.xacro"/>
-  <xacro:include filename="$(find rrbot_description)/urdf/gazebo_physics.xacro"/>
   <xacro:include filename="$(find rrbot_description)/urdf/gazebo_plugins.xacro"/>
   <!-- Used for fixing robot to Gazebo 'base_link' -->
@@ -34,60 +33,4 @@
     </inertial>
   </link>
-  <joint name="joint1" type="continuous">
-    <parent link="link1"/>
-    <child link="link2"/>
-    <origin xyz="0 ${width} ${height1 - axel_offset}" rpy="0 0 0"/>
-    <axis xyz="0 1 0"/>
-    <dynamics damping="0.7"/>
-  </joint>
-  <!-- Middle Link -->
-  <link name="link2">
-    <collision>
-      <origin xyz="0 0 ${height2/2 - axel_offset}" rpy="0 0 0"/>
-      <geometry>
-	<box size="${width} ${width} ${height2}"/>
-      </geometry>
-    </collision>
-    <visual>
-      <origin xyz="0 0 ${height2/2 - axel_offset}" rpy="0 0 0"/>
-      <geometry>
-	<box size="${width} ${width} ${height2}"/>
-      </geometry>
-      <material name="orange"/>
-    </visual>
-    <inertial>
-      <origin xyz="0 0 ${height2/2 - axel_offset}" rpy="0 0 0"/>
-      <mass value="${mass}"/>
-      <xacro:box_inertia mass="${mass}" width="${width}" height="${height2}" />
-    </inertial>
-  </link>
-  <joint name="joint2" type="continuous">
-    <parent link="link2"/>
-    <child link="link3"/>
-    <origin xyz="0 ${width} ${height2 - axel_offset*2}" rpy="0 0 0"/>
-    <axis xyz="0 1 0"/>
-    <dynamics damping="0.7"/>
-  </joint>
-  <!-- Top Link -->
-  <link name="link3">
-    <collision>
-      <origin xyz="0 0 ${height3/2 - axel_offset}" rpy="0 0 0"/>
-      <geometry>
-	<box size="${width} ${width} ${height3}"/>
-      </geometry>
-    </collision>
-    <visual>
-      <origin xyz="0 0 ${height3/2 - axel_offset}" rpy="0 0 0"/>
-      <geometry>
-	<box size="${width} ${width} ${height3}"/>
-      </geometry>
-      <material name="orange"/>
-    </visual>
-    <inertial>
-      <origin xyz="0 0 ${height3/2 - axel_offset}" rpy="0 0 0"/>
-      <mass value="${mass}"/>
-      <xacro:box_inertia mass="${mass}" width="${width}" height="${height3}" />
-    </inertial>
-  </link>
   <joint name="camera_joint" type="fixed">
     <axis xyz="0 1 0" />
@@ -99,15 +42,15 @@
   <link name="camera_link">
     <collision>
-      <origin xyz="0 0 ${height2}" rpy="0 0.5 0"/>
+      <origin xyz="0 0 ${height2}" rpy="0 -0.95 0"/>
       <geometry>
-	<box size="${camera_link} ${camera_link} ${camera_link}"/>
+	<cylinder radius="${camera_link}" length="${camera_link*2}"/>
       </geometry>
     </collision>
     <visual>
-      <origin xyz="0 0 ${height2}" rpy="0 0.5 0"/>
+      <origin xyz="0 0 ${height2}" rpy="0 -0.95 0"/>
       <geometry>
-	<box size="${camera_link} ${camera_link} ${camera_link}"/>
+	<cylinder radius="${camera_link}" length="${camera_link*2}"/>
       </geometry>
-      <material name="red"/>
+      <material name="grey"/>
     </visual>
     <inertial>
